File: NomadBall44_R/NomadBall44_R.kicad_sch (KiCad schematic)
At the start: 48 parts, among them SW1 SW_Push, SW10 SW_Push, SW11 SW_Push, SW12 SW_Push, SW13 SW_Push, SW14 SW_Push, SW15 SW_Push, SW16 SW_Push, SW17 SW_Push, SW18 SW_Push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

Commit message: マイコンまわりの配線が完了 & ラベルの間違えを修正
Connections:
- net Row2: no longer U1.8 (P1.12_D7_RX)
- net Row3: now also U1.8 (P1.12_D7_RX)
Changed lines of the file:
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@@
 		)
 	)
-	(global_label "Row2"
+	(global_label "Row3"
 		(shape input)
 		(at 80.01 53.34 0)
