File: NomadBall44_L/NomadBall44_L.kicad_sch (KiCad schematic)
At the start: 48 parts, among them SW1 SW_Push, SW10 SW_Push, SW11 SW_Push, SW12 SW_Push, SW13 SW_Push, SW14 SW_Push, SW15 SW_Push, SW16 SW_Push, SW17 SW_Push, SW18 SW_Push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

Commit message: 左手用の回路図を作成
Parts:
- removed J1: ~, NomadBall44:pmw3610_connector, symbol NomadBall44:pmw3610_breakout
- removed SW21: RotaryEncoder_Switch, Rotary_Encoder:RotaryEncoder_Alps_EC12E-Switch_Vertical_H20mm, symbol Device:RotaryEncoder_Switch
- added D23: D, NomadBall44:Diode_SMD, symbol Device:D
- added SW21: SW_Push, NomadBall44:Kailh_Choc_V1_Hotswap_thin_via, symbol Switch:SW_Push
- added SW23: SW_Push, NomadBall44:Choc_v2_Hotswap_1u, symbol Switch:SW_Push
- renumbered SW23 to SW24
Connections:
- net Col2: now also SW21.1
- net Col4: now also SW23.1
- net Row3: now also D23.1 (K)
- net at D21.2 (A): now also SW21.2
- net 3.3V: no longer names the net of U1.12 (3V3)
- net CS: no longer names the net of U1.3 (P0.28_A2_D2)
- net MOTION: no longer names the net of U1.4 (P0.29_A3_D3)
- net RE_A: no longer names the net of U1.5 (P0.04_A4_D4_SDA)
- net RE_B: no longer names the net of U1.6 (P0.05_A5_D5_SCL)
- net SCLK: no longer names the net of U1.2 (P0.03_A1_D1)
- net SDIO: no longer names the net of U1.1 (P0.02_A0_D0)
- new net: D23.2 (A), SW23.2
- no-connect marks 10 -> 16

Commit message: フットプリントの割り当てを更新
Parts:
- U1: footprint NomadBall44:XIAO-nRF52840-Plus -> NomadBall44:XIAO-nRF52840-Plus-ver2
Changed lines of the file:
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@@
 			)
 		)
-		(property "Footprint" "NomadBall44:XIAO-nRF52840-Plus"
+		(property "Footprint" "NomadBall44:XIAO-nRF52840-Plus-ver2"
 			(at 56.388 48.26 0)
 			(effects
