File: NomadBall44_R_Bottom/NomadBall44_R_Bottom.kicad_pcb (KiCad board)
At the start: 2 copper layers, 147.4 x 87.5 mm, 13 parts

Commit message: ボトムプレートのガーバファイルを生成
Parts:
- removed BT1: Battery_Cell, NomadBall44:JST_S2B-PH-SM4-TB
- removed J1: ~, NomadBall44:pmw3610_connector
