File: pmw3610_breakout/pmw3610_breakout.kicad_sch (KiCad schematic)
At the start: 13 parts, among them J1 Conn_01x08, U1 MCP1700T-1802E/TT, U2 PMW3610

Commit message: 抵抗が大きすぎたので修正
Parts:
- R1: value 2M -> 10k
Changed lines of the file:
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@@
 			)
 		)
-		(property "Value" "2M"
+		(property "Value" "10k"
 			(at 114.554 120.142 90)
 			(effects
