File: pmw3610_breakout/pmw3610_breakout.kicad_pcb (KiCad board)
At the start: 2 copper layers, 22 x 23.5 mm, 13 parts, among them J1 Conn_01x08, U1 MCP1700T-1802E/TT, U2 PMW3610

Commit message: 抵抗が大きすぎたので修正
Parts:
- R1: value 2M -> 10k
Changed lines of the file:
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@@
 			)
 		)
-		(property "Value" "2M"
+		(property "Value" "10k"
 			(at 0 -1.43 180)
 			(layer "B.Fab")
@@
 			)
 		)
-		(property "LCSC" "C22976"
+		(property "LCSC" "C25804"
 			(at 0 0 0)
 			(layer "B.SilkS")

Commit message: 抵抗値を微修正
Parts:
- C5: value 100n (X7R) -> 100n
- C7: value 10n (X7R) -> 10n
Changed lines of the file:
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@@
 			)
 		)
-		(property "Value" " 10n (X7R)"
+		(property "Value" "10n"
 			(at 0 -1.43 180)
 			(layer "B.Fab")
@@
 			)
 		)
-		(property "Value" " 100n (X7R)"
+		(property "Value" "100n"
 			(at 0 -1.43 180)
 			(layer "B.Fab")
