File: design_data/NomadBall44_L_v2/NomadBall44_L_v2.kicad_sch (KiCad schematic)
At the start: 49 parts, among them SW1 SW_Push, SW10 SW_Push, SW11 SW_Push, SW12 SW_Push, SW13 SW_Push, SW14 SW_Push, SW15 SW_Push, SW16 SW_Push, SW17 SW_Push, SW18 SW_Push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

Commit message: シンボルとフットプリントの紐付けを修正
Parts:
- SW19, SW20, SW21: footprint NomadBall44:Kailh_Choc_V1_Hotswap_thin_via -> NomadBall44:Choc_v2_Hotswap_1u
- U1: footprint NomadBall44:XIAO-nRF52840-Plus-ver2 -> NomadBall44:XIAO-nRF52840-Plus-ver3
Changed lines of the file:
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@@
 			)
 		)
-		(property "Footprint" "NomadBall44:Kailh_Choc_V1_Hotswap_thin_via"
+		(property "Footprint" "NomadBall44:Choc_v2_Hotswap_1u"
 			(at 116.84 83.82 0)
 			(effects
@@
 			)
 		)
-		(property "Footprint" "NomadBall44:XIAO-nRF52840-Plus-ver2"
+		(property "Footprint" "NomadBall44:XIAO-nRF52840-Plus-ver3"
 			(at 56.388 48.26 0)
 			(effects
@@
 			)
 		)
-		(property "Footprint" "NomadBall44:Kailh_Choc_V1_Hotswap_thin_via"
+		(property "Footprint" "NomadBall44:Choc_v2_Hotswap_1u"
 			(at 135.89 83.82 0)
 			(effects
@@
 			)
 		)
-		(property "Footprint" "NomadBall44:Kailh_Choc_V1_Hotswap_thin_via"
+		(property "Footprint" "NomadBall44:Choc_v2_Hotswap_1u"
 			(at 154.94 83.82 0)
 			(effects
