File: design_data/NomadBall44_L_v2/NomadBall44_L_v2.kicad_pcb (KiCad board)
At the start: 2 copper layers, 149 x 96.5 mm, 57 parts, among them SW1 SW_Push, SW10 SW_Push, SW11 SW_Push, SW12 SW_Push, SW13 SW_Push, SW14 SW_Push, SW15 SW_Push, SW16 SW_Push, SW17 SW_Push, SW18 SW_Push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

Commit message: gndの塗りつぶしを実行
Routing:
- added copper zone on B.Cu, net GND
- added copper zone on F.Cu, net GND
Changed lines of the file:
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@@
 		(net 37)
+	)
+	(zone
+		(net 37)
+		(net_name "GND")
+		(layers "F.Cu" "B.Cu")
+		(hatch edge 0.5)
+		(connect_pads
+			(clearance 0.5)
+		)
+		(min_thickness 0.25)
+		(filled_areas_thickness no)
+		(fill yes
+			(thermal_gap 0.5)
+			(thermal_bridge_width 0.5)
+		)
+		(polygon
+			(pts
+				(xy 247.71 51.74) (xy 127.53 52.29) (xy 128.09 155.78) (xy 282.05 156.22) (xy 282.3 51.65) (xy 247.65 51.74)
+				(xy 247.64 51.74)
+			)
+		)
 	)
 	(embedded_fonts no)
