File: design_data/NomadBall44_L_Top_v2/NomadBall44_L_Top_v2.kicad_pcb (KiCad board)
At the start: 2 copper layers, 116.7 x 81.5 mm, 26 parts, among them SW1 SW_Push, SW10 SW_Push, SW11 SW_Push, SW12 SW_Push, SW13 SW_Push, SW14 SW_Push, SW15 SW_Push, SW16 SW_Push, SW17 SW_Push, SW18 SW_Push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

Commit message: トッププレートのネジ穴フットプリントを変更
Parts:
- REF** (x6): footprint NomadBall44:m2_Screw_Hole_EdgeCuts -> NomadBall44:m2_Screw_Hole
Changed lines of the file:
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@@
 		(embedded_fonts no)
 	)
-	(footprint "NomadBall44:m2_Screw_Hole_EdgeCuts"
+	(footprint "NomadBall44:m2_Screw_Hole"
 		(layer "F.Cu")
 		(at 152.664757 111.959999)
@@
 			(at 0 -3.2 0)
 			(layer "F.Fab")
-			(hide yes)
 			(effects
 				(font
@@
 			(at 0 3.2 0)
 			(layer "F.Fab")
-			(hide yes)
 			(effects
 				(font
@@
 		(fp_circle
 			(center 0 0)
-			(end 1.1 0)
-			(stroke
-				(width 0.01)
+			(end 2.2 0)
+			(stroke
+				(width 0.15)
 				(type solid)
 			)
 			(fill no)
-			(layer "Edge.Cuts")
+			(layer "Cmts.User")
+		)
+		(fp_circle
+			(center 0 0)
+			(end 2.45 0)
+			(stroke
+				(width 0.05)
+				(type solid)
+			)
+			(fill no)
+			(layer "F.CrtYd")
 		)
 		(fp_text user "${REFERENCE}"
-			(at 0 0 0)
-			(layer "F.Fab")
-			(effects
-				(font
-					(size 1 1)
-					(thickness 0.15)
-				)
-			)
+			(at 0.3 0 0)
+			(layer "F.Fab")
+			(effects
+				(font
+					(size 1 1)
+					(thickness 0.15)
+				)
+			)
+		)
+		(pad "" np_thru_hole circle
+			(at 0 0)
+			(size 2.2 2.2)
+			(drill 2.2)
+			(layers "*.Cu" "*.Mask")
 		)
 		(embedded_fonts no)
@@
 		(embedded_fonts no)
 	)
-	(footprint "NomadBall44:m2_Screw_Hole_EdgeCuts"
+	(footprint "NomadBall44:m2_Screw_Hole"
 		(layer "F.Cu")
 		(at 230.714757 78.349999)
@@
 			(at 0 -3.2 0)
 			(layer "F.Fab")
-			(hide yes)
 			(effects
 				(font
@@
 			(at 0 3.2 0)
 			(layer "F.Fab")
-			(hide yes)
 			(effects
 				(font
@@
 		(fp_circle
 			(center 0 0)
-			(end 1.1 0)
-			(stroke
-				(width 0.01)
+			(end 2.2 0)
+			(stroke
+				(width 0.15)
 				(type solid)
 			)
 			(fill no)
-			(layer "Edge.Cuts")
+			(layer "Cmts.User")
+		)
+		(fp_circle
+			(center 0 0)
+			(end 2.45 0)
+			(stroke
+				(width 0.05)
+				(type solid)
+			)
+			(fill no)
+			(layer "F.CrtYd")
 		)
 		(fp_text user "${REFERENCE}"
-			(at 0 0 0)
-			(layer "F.Fab")
-			(effects
-				(font
-					(size 1 1)
-					(thickness 0.15)
-				)
-			)
+			(at 0.3 0 0)
+			(layer "F.Fab")
+			(effects
+				(font
+					(size 1 1)
+					(thickness 0.15)
+				)
+			)
+		)
+		(pad "" np_thru_hole circle
+			(at 0 0)
+			(size 2.2 2.2)
+			(drill 2.2)
+			(layers "*.Cu" "*.Mask")
 		)
 		(embedded_fonts no)
 	)
-	(footprint "NomadBall44:m2_Screw_Hole_EdgeCuts"
+	(footprint "NomadBall44:m2_Screw_Hole"
 		(layer "F.Cu")
 		(at 190.98 62.67)
@@
 			(at 0 -3.2 0)
 			(layer "F.Fab")
-			(hide yes)
 			(effects
 				(font
@@
 			(at 0 3.2 0)
 			(layer "F.Fab")
-			(hide yes)
 			(effects
 				(font
@@
 		(fp_circle
 			(center 0 0)
-			(end 1.1 0)
-			(stroke
-				(width 0.01)
+			(end 2.2 0)
+			(stroke
+				(width 0.15)
 				(type solid)
 			)
 			(fill no)
-			(layer "Edge.Cuts")
+			(layer "Cmts.User")
+		)
+		(fp_circle
+			(center 0 0)
+			(end 2.45 0)
+			(stroke
+				(width 0.05)
+				(type solid)
+			)
+			(fill no)
+			(layer "F.CrtYd")
 		)
 		(fp_text user "${REFERENCE}"
-			(at 0 0 0)
-			(layer "F.Fab")
-			(effects
-				(font
-					(size 1 1)
-					(thickness 0.15)
-				)
-			)
+			(at 0.3 0 0)
+			(layer "F.Fab")
+			(effects
+				(font
+					(size 1 1)
+					(thickness 0.15)
+				)
+			)
+		)
+		(pad "" np_thru_hole circle
+			(at 0 0)
+			(size 2.2 2.2)
+			(drill 2.2)
+			(layers "*.Cu" "*.Mask")
 		)
 		(embedded_fonts no)
@@
 		(embedded_fonts no)
 	)
-	(footprint "NomadBall44:m2_Screw_Hole_EdgeCuts"
+	(footprint "NomadBall44:m2_Screw_Hole"
 		(layer "F.Cu")
 		(at 230.724757 97.829999)
@@
 			(at 0 -3.2 0)
 			(layer "F.Fab")
-			(hide yes)
 			(effects
 				(font
@@
 			(at 0 3.2 0)
 			(layer "F.Fab")
-			(hide yes)
 			(effects
 				(font
@@
 		(fp_circle
 			(center 0 0)
-			(end 1.1 0)
-			(stroke
-				(width 0.01)
+			(end 2.2 0)
+			(stroke
+				(width 0.15)
 				(type solid)
 			)
 			(fill no)
-			(layer "Edge.Cuts")
+			(layer "Cmts.User")
+		)
+		(fp_circle
+			(center 0 0)
+			(end 2.45 0)
+			(stroke
+				(width 0.05)
+				(type solid)
+			)
+			(fill no)
+			(layer "F.CrtYd")
 		)
 		(fp_text user "${REFERENCE}"
-			(at 0 0 0)
-			(layer "F.Fab")
-			(effects
-				(font
-					(size 1 1)
-					(thickness 0.15)
-				)
-			)
+			(at 0.3 0 0)
+			(layer "F.Fab")
+			(effects
+				(font
+					(size 1 1)
+					(thickness 0.15)
+				)
+			)
+		)
+		(pad "" np_thru_hole circle
+			(at 0 0)
+			(size 2.2 2.2)
+			(drill 2.2)
+			(layers "*.Cu" "*.Mask")
 		)
 		(embedded_fonts no)
 	)
-	(footprint "NomadBall44:m2_Screw_Hole_EdgeCuts"
+	(footprint "NomadBall44:m2_Screw_Hole"
 		(layer "F.Cu")
 		(at 190.98 119.59)
@@
 			(at 0 -3.2 0)
 			(layer "F.Fab")
-			(hide yes)
 			(effects
 				(font
@@
 			(at 0 3.2 0)
 			(layer "F.Fab")
-			(hide yes)
 			(effects
 				(font
@@
 		(fp_circle
 			(center 0 0)
-			(end 1.1 0)
-			(stroke
-				(width 0.01)
+			(end 2.2 0)
+			(stroke
+				(width 0.15)
 				(type solid)
 			)
 			(fill no)
-			(layer "Edge.Cuts")
+			(layer "Cmts.User")
+		)
+		(fp_circle
+			(center 0 0)
+			(end 2.45 0)
+			(stroke
+				(width 0.05)
+				(type solid)
+			)
+			(fill no)
+			(layer "F.CrtYd")
 		)
 		(fp_text user "${REFERENCE}"
-			(at 0 0 0)
-			(layer "F.Fab")
-			(effects
-				(font
-					(size 1 1)
-					(thickness 0.15)
-				)
-			)
+			(at 0.3 0 0)
+			(layer "F.Fab")
+			(effects
+				(font
+					(size 1 1)
+					(thickness 0.15)
+				)
+			)
+		)
+		(pad "" np_thru_hole circle
+			(at 0 0)
+			(size 2.2 2.2)
+			(drill 2.2)
+			(layers "*.Cu" "*.Mask")
 		)
 		(embedded_fonts no)
@@
 		(embedded_fonts no)
 	)
-	(footprint "NomadBall44:m2_Screw_Hole_EdgeCuts"
+	(footprint "NomadBall44:m2_Screw_Hole"
 		(layer "F.Cu")
 		(at 152.724757 85.089999)
@@
 			(at 0 -3.2 0)
 			(layer "F.Fab")
-			(hide yes)
 			(effects
 				(font
@@
 			(at 0 3.2 0)
 			(layer "F.Fab")
-			(hide yes)
 			(effects
 				(font
@@
 		(fp_circle
 			(center 0 0)
-			(end 1.1 0)
-			(stroke
-				(width 0.01)
+			(end 2.2 0)
+			(stroke
+				(width 0.15)
 				(type solid)
 			)
 			(fill no)
-			(layer "Edge.Cuts")
+			(layer "Cmts.User")
+		)
+		(fp_circle
+			(center 0 0)
+			(end 2.45 0)
+			(stroke
+				(width 0.05)
+				(type solid)
+			)
+			(fill no)
+			(layer "F.CrtYd")
 		)
 		(fp_text user "${REFERENCE}"
-			(at 0 0 0)
-			(layer "F.Fab")
-			(effects
-				(font
-					(size 1 1)
-					(thickness 0.15)
-				)
-			)
+			(at 0.3 0 0)
+			(layer "F.Fab")
+			(effects
+				(font
+					(size 1 1)
+					(thickness 0.15)
+				)
+			)
+		)
+		(pad "" np_thru_hole circle
+			(at 0 0)
+			(size 2.2 2.2)
+			(drill 2.2)
+			(layers "*.Cu" "*.Mask")
 		)
 		(embedded_fonts no)
